Commit message: clean for milestone 2

File: body.urdf (robot description, URDF)
Before this commit: robot robot, 9 links, 8 joints
Links:
- removed link LeftLeg
- removed link LeftLowerLeg
- removed link RightLeg
- removed link RightLowerLeg
- link Torso: geometry collision box size=0.5 1 1; visual box size=0.5 1 1
Joints:
- removed joint LeftLeg_LeftLowerLeg
- removed joint RightLeg_RightLowerLeg
- removed joint Torso_LeftLeg
- removed joint Torso_RightLeg

Commit message: robot body made, fitness function goofy

File: body.urdf (robot description, URDF)
Before this commit: robot robot, 5 links, 4 joints
Links:
- added link BackFoot, mass 1; collision box size=1 0.75 0.25; visual box size=1 0.75 0.25
- added link FrontFoot, mass 1; collision box size=1 0.75 0.25; visual box size=1 0.75 0.25
- link BackLeg: geometry collision box size=0.25 0.25 1; visual box size=0.25 0.25 1
- link BackLowerLeg: geometry collision box size=0.25 0.25 1; visual box size=0.25 0.25 1
- link FrontLeg: geometry collision box size=0.25 0.25 1; visual box size=0.25 0.25 1
- link FrontLowerLeg: geometry collision box size=0.25 0.25 1; visual box size=0.25 0.25 1
Joints:
- added joint BackLowerLeg_BackFoot: type revolute, parent BackLowerLeg, child BackFoot, origin xyz=0 0 -1 rpy=0 0 0, axis 0 1 0, limit lower=-3.14159 upper=3.14159 effort=0.0 velocity=0.0
- added joint FrontLowerLeg_FrontFoot: type revolute, parent FrontLowerLeg, child FrontFoot, origin xyz=0 0 -1 rpy=0 0 0, axis 0 1 0, limit lower=-3.14159 upper=3.14159 effort=0.0 velocity=0.0
- joint BackLeg_BackLowerLeg: axis 1 0 0 -> 0 1 0; origin xyz=0 -1 0 rpy=0 0 0 -> xyz=0 0 -1 rpy=0 0 0
- joint FrontLeg_FrontLowerLeg: axis 1 0 0 -> 0 1 0; origin xyz=0 1 0 rpy=0 0 0 -> xyz=0 0 -1 rpy=0 0 0
- joint Torso_BackLeg: axis 1 0 0 -> 0 1 0; origin xyz=0 -0.5 1 rpy=0 0 0 -> xyz=0 -0.5 3.0 rpy=0 0 0
- joint Torso_FrontLeg: axis 1 0 0 -> 0 1 0; origin xyz=0 0.5 1 rpy=0 0 0 -> xyz=0 0.5 3.0 rpy=0 0 0

Commit message: quadruped

File: body.urdf (robot description, URDF)
Before this commit: robot robot, 5 links, 4 joints
Links:
- added link LeftLeg, mass 1; collision box size=1 0.2 0.2; visual box size=1 0.2 0.2
- added link LeftLowerLeg, mass 1; collision box size=0.2 0.2 1; visual box size=0.2 0.2 1
- added link RightLeg, mass 1; collision box size=1 0.2 0.2; visual box size=1 0.2 0.2
- added link RightLowerLeg, mass 1; collision box size=0.2 0.2 1; visual box size=0.2 0.2 1
Joints:
- added joint LeftLeg_LeftLowerLeg: type revolute, parent LeftLeg, child LeftLowerLeg, origin xyz=-1 0 0 rpy=0 0 0, axis 0 1 0, limit lower=-3.14159 upper=3.14159 effort=0.0 velocity=0.0
- added joint RightLeg_RightLowerLeg: type revolute, parent RightLeg, child RightLowerLeg, origin xyz=1 0 0 rpy=0 0 0, axis 0 1 0, limit lower=-3.14159 upper=3.14159 effort=0.0 velocity=0.0
- added joint Torso_LeftLeg: type revolute, parent Torso, child LeftLeg, origin xyz=-0.5 0 1 rpy=0 0 0, axis 0 1 0, limit lower=-3.14159 upper=3.14159 effort=0.0 velocity=0.0
- added joint Torso_RightLeg: type revolute, parent Torso, child RightLeg, origin xyz=0.5 0 1 rpy=0 0 0, axis 0 1 0, limit lower=-3.14159 upper=3.14159 effort=0.0 velocity=0.0

Commit message: bipedal final project

File: body.urdf (robot description, URDF)
Before this commit: robot robot, 7 links, 6 joints
Links:
- added link LeftArm, mass 1; collision box size=1 0.25 0.25; visual box size=1 0.25 0.25
- added link RightArm, mass 1; collision box size=1 0.25 0.25; visual box size=1 0.25 0.25
- link BackFoot: geometry collision box size=1.25 0.75 0.25; visual box size=1.25 0.75 0.25
- link BackLeg: geometry collision box size=1 0.25 0.25; visual box size=1 0.25 0.25
- link FrontFoot: geometry collision box size=1.25 0.75 0.25; visual box size=1.25 0.75 0.25
- link FrontLeg: geometry collision box size=1 0.25 0.25; visual box size=1 0.25 0.25
Joints:
- added joint Torso_LeftArm: type revolute, parent Torso, child LeftArm, origin xyz=0 -0.5 1.75 rpy=0 0 0, axis 0 1 0, limit lower=-3.14159 upper=3.14159 effort=0.0 velocity=0.0
- added joint Torso_RightArm: type revolute, parent Torso, child RightArm, origin xyz=0 0.5 1.75 rpy=0 0 0, axis 0 1 0, limit lower=-3.14159 upper=3.14159 effort=0.0 velocity=0.0
- joint BackLeg_BackLowerLeg: origin xyz=0 0 -1 rpy=0 0 0 -> xyz=1 0 0 rpy=0 0 0
- joint FrontLeg_FrontLowerLeg: origin xyz=0 0 -1 rpy=0 0 0 -> xyz=1 0 0 rpy=0 0 0
- joint Torso_BackLeg: origin xyz=0 -0.5 3.0 rpy=0 0 0 -> xyz=0 -0.5 1.25 rpy=0 0 0
- joint Torso_FrontLeg: origin xyz=0 0.5 3.0 rpy=0 0 0 -> xyz=0 0.5 1.25 rpy=0 0 0

Commit message: biped in trouble

File: body.urdf (robot description, URDF)
Before this commit: robot robot, 9 links, 8 joints
Links:
- removed link LeftArm
- removed link RightArm
- added link LeftFist, mass 1; collision box size=0.5 0.5 0.5; visual box size=0.5 0.5 0.5
- added link LeftUpperArm, mass 1; collision box size=0.25 0.25 1; visual box size=0.25 0.25 1
- added link RightFist, mass 1; collision box size=0.5 0.5 0.5; visual box size=0.5 0.5 0.5
- added link RightUpperArm, mass 1; collision box size=0.25 0.25 1; visual box size=0.25 0.25 1
Joints:
- removed joint Torso_LeftArm
- removed joint Torso_RightArm
- added joint LeftUpperArm_LeftFist: type revolute, parent LeftUpperArm, child LeftFist, origin xyz=0 0 -1 rpy=0 0 0, axis 0 1 0, limit lower=-3.14159 upper=3.14159 effort=0.0 velocity=0.0
- added joint RightUpperArm_RightFist: type revolute, parent RightUpperArm, child RightFist, origin xyz=0 0 -1 rpy=0 0 0, axis 0 1 0, limit lower=-3.14159 upper=3.14159 effort=0.0 velocity=0.0
- added joint Torso_LeftUpperArm: type revolute, parent Torso, child LeftUpperArm, origin xyz=0 -1 1.75 rpy=0 0 0, axis 0 1 0, limit lower=-3.14159 upper=3.14159 effort=0.0 velocity=0.0
- added joint Torso_RightUpperArm: type revolute, parent Torso, child RightUpperArm, origin xyz=0 1 1.75 rpy=0 0 0, axis 0 1 0, limit lower=-3.14159 upper=3.14159 effort=0.0 velocity=0.0
- joint Torso_BackLeg: origin xyz=0 -0.5 1.25 rpy=0 0 0 -> xyz=-0.25 -0.5 1.25 rpy=0 0 0
- joint Torso_FrontLeg: origin xyz=0 0.5 1.25 rpy=0 0 0 -> xyz=-0.25 0.5 1.25 rpy=0 0 0

Commit message: Biped performs a small jump

File: body.urdf (robot description, URDF)
Before this commit: robot robot, 11 links, 10 joints
Links:
- link BackLeg: geometry collision box size=0.25 0.25 1; visual box size=0.25 0.25 1
- link FrontLeg: geometry collision box size=0.25 0.25 1; visual box size=0.25 0.25 1
Joints:
- joint BackLeg_BackLowerLeg: origin xyz=1 0 0 rpy=0 0 0 -> xyz=0 0 -1 rpy=0 0 0
- joint FrontLeg_FrontLowerLeg: origin xyz=1 0 0 rpy=0 0 0 -> xyz=0 0 -1 rpy=0 0 0
- joint Torso_BackLeg: origin xyz=-0.25 -0.5 1.25 rpy=0 0 0 -> xyz=0 -0.5 2.25 rpy=0 0 0
- joint Torso_FrontLeg: origin xyz=-0.25 0.5 1.25 rpy=0 0 0 -> xyz=0 0.5 2.25 rpy=0 0 0
- joint Torso_LeftUpperArm: origin xyz=0 -1 1.75 rpy=0 0 0 -> xyz=0 -1 2.75 rpy=0 0 0
- joint Torso_RightUpperArm: origin xyz=0 1 1.75 rpy=0 0 0 -> xyz=0 1 2.75 rpy=0 0 0

Commit message: FInished BIPED

File: body.urdf (robot description, URDF)
Before this commit: robot robot, 11 links, 10 joints
Links:
- removed link LeftFist
- removed link RightFist
- link BackFoot: geometry collision box size=0.8 0.8 0.2; visual box size=0.8 0.8 0.2
- link BackLeg: geometry collision box size=0.2 0.2 0.8; visual box size=0.2 0.2 0.8
- link BackLowerLeg: geometry collision box size=0.2 0.2 0.8; visual box size=0.2 0.2 0.8
- link FrontFoot: geometry collision box size=0.8 0.8 0.2; visual box size=0.8 0.8 0.2
- link FrontLeg: geometry collision box size=0.2 0.2 0.8; visual box size=0.2 0.2 0.8
- link FrontLowerLeg: geometry collision box size=0.2 0.2 0.8; visual box size=0.2 0.2 0.8
- link LeftUpperArm: geometry collision box size=1 0.2 0.2; visual box size=1 0.2 0.2
- link RightUpperArm: geometry collision box size=1 0.2 0.2; visual box size=1 0.2 0.2
- link Torso: geometry collision box size=0.5 1 0.5; visual box size=0.5 1 0.5
Joints:
- removed joint LeftUpperArm_LeftFist
- removed joint RightUpperArm_RightFist
- joint BackLeg_BackLowerLeg: origin xyz=0 0 -1 rpy=0 0 0 -> xyz=0 0 -0.8 rpy=0 0 0
- joint BackLowerLeg_BackFoot: origin xyz=0 0 -1 rpy=0 0 0 -> xyz=0 0 -0.9 rpy=0 0 0
- joint FrontLeg_FrontLowerLeg: origin xyz=0 0 -1 rpy=0 0 0 -> xyz=0 0 -0.8 rpy=0 0 0
- joint FrontLowerLeg_FrontFoot: origin xyz=0 0 -1 rpy=0 0 0 -> xyz=0 0 -0.9 rpy=0 0 0
- joint Torso_BackLeg: origin xyz=0 -0.5 2.25 rpy=0 0 0 -> xyz=0 -0.5 1.8 rpy=0 0 0
- joint Torso_FrontLeg: origin xyz=0 0.5 2.25 rpy=0 0 0 -> xyz=0 0.5 1.8 rpy=0 0 0
- joint Torso_LeftUpperArm: origin xyz=0 -1 2.75 rpy=0 0 0 -> xyz=0.5 -0.5 2.3 rpy=0 0 0
- joint Torso_RightUpperArm: origin xyz=0 1 2.75 rpy=0 0 0 -> xyz=0.5 0.5 2.3 rpy=0 0 0
